File: KiCad/ByggernProject (2).kicad_sch (KiCad schematic)
At the start: 28 parts, among them J1 AVR-JTAG-10, J2 AVR-JTAG-10, SW1 SW_Push, SW2 SW_Push, U1 LATCH, U2 L7805, U3 MAX232, U5 SRAM, U6 ATmega162-16P, U7 MAX232, U9 ATmega162-16P

Commit message: Kicad with wires on MCP2515
Parts:
- added U4, U8: MCP2515-xSO, Package_SO:SOIC-18W_7.5x11.6mm_P1.27mm, symbol Interface_CAN_LIN:MCP2515-xSO
Connections:
- net +5V: now also ADC1.22 (VDD), U4.18 (VDD), U8.18 (VDD)
- net GND: now also U4.9 (VSS), U8.9 (VSS); no longer U9.20 (GND)
- net SCK PB7: now reaches OLED_Controller. (DISP_RES)
- net SCK PB7: now also U9.8 (PB7), U8.13 (SCK)
- net CS PB4 Board: now reaches OLED_Controller. (DISP_RES), U9.5 (PB4)
- net CS PB4 Board: now also U8.16 (~{CS})
- net MOSI PB5: now reaches OLED_Controller. (DISP_RES), U9.7 (PB6)
- net MOSI PB5: now also U8.14 (SI)
- net at SW2.2, U9.9 (~{RESET}): now also U8.17 (~{RESET})
- net CAN INT PD3: now reaches U9.13 (PD3)
- net CAN INT PD3: now also U8.12 (~{INT})
- net at U9.3 (PB2): now also OLED_Controller. (DISP_RES)
- net CS PB3 Disp: now reaches U9.4 (PB3)
- net CS PB3 Disp: now also OLED_Controller. (DISP_RES)
- net PB6_MISO renamed MISO PB6
- net MISO PB6: now also U8.15 (SO)
- new net CLK 4.9MHz: U8.7 (OSC2), U8.8 (OSC1)
