File: KiCad/ByggernProject.kicad_sch (KiCad schematic)
At the start: 28 parts, among them J1 AVR-JTAG-10, J2 AVR-JTAG-10, SW1 SW_Push, SW2 SW_Push, U1 LATCH, U2 L7805, U3 MAX232, U5 SRAM, U6 ATmega162-16P, U7 MAX232, U9 ATmega162-16P

Commit message: Add files via upload
Other:
- note added: "Pulled Up = D[7:0] is data, Pulled Down = Teansfer data to Command Register. I2C: SA0, PB2"
- note added: "RESET = Pulled Up, Chip enable = Pull Down, Connect to MCU, PB3"
- note added: "Slave Select, PB4"
- note removed: "Pulled Up = D[7:0] is data, Pulled Down = Teansfer data to Command Register. I2C: SA0"
- note removed: "RESET = Pulled Up, Chip enable = Pull Down, Connect to MCU"
- note removed: "Slave Select"
Changed lines of the file:
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@@
 		)
 	)
-	(text "Pulled Up = D[7:0] is data, Pulled Down = Teansfer data to Command Register. I2C: SA0"
+	(text "Pulled Up = D[7:0] is data, Pulled Down = Teansfer data to Command Register. I2C: SA0, PB2\n"
 		(exclude_from_sim no)
 		(at 666.242 91.186 0)
@@
 		)
 	)
-	(text "Slave Select"
+	(text "Slave Select, PB4"
 		(exclude_from_sim no)
 		(at 631.952 99.06 0)
@@
 		)
 	)
-	(text "RESET = Pulled Up, Chip enable = Pull Down, Connect to MCU\n"
+	(text "RESET = Pulled Up, Chip enable = Pull Down, Connect to MCU, PB3\n\n"
 		(exclude_from_sim no)
 		(at 653.288 94.996 0)
@@
 		)
 		(instances
-			(project "ByggernProject"
+			(project "ByggernProject (2)"
 				(path "/43741492-b21a-4f5a-8ce1-a54a4b312e32"
 					(reference "U1")
@@
 		)
 		(instances
-			(project "ByggernProject"
+			(project "ByggernProject (2)"
 				(path "/43741492-b21a-4f5a-8ce1-a54a4b312e32"
 					(reference "C7")
@@
 		)
 		(instances
-			(project "ByggernProject"
+			(project "ByggernProject (2)"
 				(path "/43741492-b21a-4f5a-8ce1-a54a4b312e32"
 					(reference "#PWR014")
@@
 		)
 		(instances
-			(project "ByggernProject"
+			(project "ByggernProject (2)"
 				(path "/43741492-b21a-4f5a-8ce1-a54a4b312e32"
 					(reference "1k")
@@
 		)
 		(instances
-			(project "ByggernProject"
+			(project "ByggernProject (2)"
 				(path "/43741492-b21a-4f5a-8ce1-a54a4b312e32"
 					(reference "SW1")
@@
 		)
 		(instances
-			(project "ByggernProject"
+			(project "ByggernProject (2)"
 				(path "/43741492-b21a-4f5a-8ce1-a54a4b312e32"
 					(reference "#PWR011")
@@
 		)
 		(instances
-			(project "ByggernProject"
+			(project "ByggernProject (2)"
 				(path "/43741492-b21a-4f5a-8ce1-a54a4b312e32"
 					(reference "#PWR021")
@@
 		)
 		(instances
-			(project "ByggernProject"
+			(project "ByggernProject (2)"
 				(path "/43741492-b21a-4f5a-8ce1-a54a4b312e32"
 					(reference "#PWR04")
@@
 		)
 		(instances
-			(project "ByggernProject"
+			(project "ByggernProject (2)"
 				(path "/43741492-b21a-4f5a-8ce1-a54a4b312e32"
 					(reference "4.7my1")
@@
 		)
 		(instances
-			(project "ByggernProject"
+			(project "ByggernProject (2)"
 				(path "/43741492-b21a-4f5a-8ce1-a54a4b312e32"
 					(reference "C2")
@@
 		)
 		(instances
-			(project "ByggernProject"
+			(project "ByggernProject (2)"
 				(path "/43741492-b21a-4f5a-8ce1-a54a4b312e32"
 					(reference "U5")
@@
 		)
 		(instances
-			(project "ByggernProject"
+			(project "ByggernProject (2)"
 				(path "/43741492-b21a-4f5a-8ce1-a54a4b312e32"
 					(reference "#PWR05")
@@
 		)
 		(instances
-			(project "ByggernProject"
+			(project "ByggernProject (2)"
 				(path "/43741492-b21a-4f5a-8ce1-a54a4b312e32"
 					(reference "J1")
@@
 		)
 		(instances
-			(project "ByggernProject"
+			(project "ByggernProject (2)"
 				(path "/43741492-b21a-4f5a-8ce1-a54a4b312e32"
 					(reference "C3")
@@
 		)
 		(instances
-			(project "ByggernProject"
+			(project "ByggernProject (2)"
 				(path "/43741492-b21a-4f5a-8ce1-a54a4b312e32"
 					(reference "PC_UART")
@@
 		)
 		(instances
-			(project "ByggernProject"
+			(project "ByggernProject (2)"
 				(path "/43741492-b21a-4f5a-8ce1-a54a4b312e32"
 					(reference "#PWR08")
@@
 		)
 		(instances
-			(project "ByggernProject"
+			(project "ByggernProject (2)"
 				(path "/43741492-b21a-4f5a-8ce1-a54a4b312e32"
 					(reference "#PWR028")
@@
 		)
 		(instances
-			(project "ByggernProject"
+			(project "ByggernProject (2)"
 				(path "/43741492-b21a-4f5a-8ce1-a54a4b312e32"
 					(reference "R2")
@@
 		)
 		(instances
-			(project "ByggernProject"
+			(project "ByggernProject (2)"
 				(path "/43741492-b21a-4f5a-8ce1-a54a4b312e32"
 					(reference "#PWR030")
@@
 		)
 		(instances
-			(project "ByggernProject"
+			(project "ByggernProject (2)"
 				(path "/43741492-b21a-4f5a-8ce1-a54a4b312e32"
 					(reference "#PWR023")
@@
 		)
 		(instances
-			(project "ByggernProject"
+			(project "ByggernProject (2)"
 				(path "/43741492-b21a-4f5a-8ce1-a54a4b312e32"
 					(reference "ADC1")
@@
 		)
 		(instances
-			(project "ByggernProject"
+			(project "ByggernProject (2)"
 				(path "/43741492-b21a-4f5a-8ce1-a54a4b312e32"
 					(reference "#PWR01")
@@
 		)
 		(instances
-			(project "ByggernProject"
+			(project "ByggernProject (2)"
 				(path "/43741492-b21a-4f5a-8ce1-a54a4b312e32"
 					(reference "#PWR02")
@@
 		)
 		(instances
-			(project "ByggernProject"
+			(project "ByggernProject (2)"
 				(path "/43741492-b21a-4f5a-8ce1-a54a4b312e32"
 					(reference "#PWR022")
@@
 		)
 		(instances
-			(project "ByggernProject"
+			(project "ByggernProject (2)"
 				(path "/43741492-b21a-4f5a-8ce1-a54a4b312e32"
 					(reference "C1")
@@
 		)
 		(instances
-			(project "ByggernProject"
+			(project "ByggernProject (2)"
 				(path "/43741492-b21a-4f5a-8ce1-a54a4b312e32"
 					(reference "#PWR026")
@@
 		)
 		(instances
-			(project "ByggernProject"
+			(project "ByggernProject (2)"
 				(path "/43741492-b21a-4f5a-8ce1-a54a4b312e32"
 					(reference "R1")
@@
 		)
 		(instances
-			(project "ByggernProject"
+			(project "ByggernProject (2)"
 				(path "/43741492-b21a-4f5a-8ce1-a54a4b312e32"
 					(reference "#PWR010")
@@
 		)
 		(instances
-			(project "ByggernProject"
+			(project "ByggernProject (2)"
 				(path "/43741492-b21a-4f5a-8ce1-a54a4b312e32"
 					(reference "0.1µ")
@@
 		)
 		(instances
-			(project "ByggernProject"
+			(project "ByggernProject (2)"
 				(path "/43741492-b21a-4f5a-8ce1-a54a4b312e32"
 					(reference "C4")
@@
 		)
 		(instances
-			(project "ByggernProject"
+			(project "ByggernProject (2)"
 				(path "/43741492-b21a-4f5a-8ce1-a54a4b312e32"
 					(reference "#PWR06")
@@
 		)
 		(instances
-			(project "ByggernProject"
+			(project "ByggernProject (2)"
 				(path "/43741492-b21a-4f5a-8ce1-a54a4b312e32"
 					(reference "#PWR09")
@@
 		)
 		(instances
-			(project "ByggernProject"
+			(project "ByggernProject (2)"
 				(path "/43741492-b21a-4f5a-8ce1-a54a4b312e32"
 					(reference "U2")
@@
 		)
 		(instances
-			(project "ByggernProject"
+			(project "ByggernProject (2)"
 				(path "/43741492-b21a-4f5a-8ce1-a54a4b312e32"
 					(reference "#PWR025")
@@
 		)
 		(instances
-			(project "ByggernProject"
+			(project "ByggernProject (2)"
 				(path "/43741492-b21a-4f5a-8ce1-a54a4b312e32"
 					(reference "#PWR03")
@@
 		)
 		(instances
-			(project "ByggernProject"
+			(project "ByggernProject (2)"
 				(path "/43741492-b21a-4f5a-8ce1-a54a4b312e32"
 					(reference "OLED_Controller")
@@
 		)
 		(instances
-			(project "ByggernProject"
+			(project "ByggernProject (2)"
 				(path "/43741492-b21a-4f5a-8ce1-a54a4b312e32"
 					(reference "#PWR029")
@@
 		)
 		(instances
-			(project "ByggernProject"
+			(project "ByggernProject (2)"
 				(path "/43741492-b21a-4f5a-8ce1-a54a4b312e32"
 					(reference "C5")
@@
 		)
 		(instances
-			(project "ByggernProject"
+			(project "ByggernProject (2)"
 				(path "/43741492-b21a-4f5a-8ce1-a54a4b312e32"
 					(reference "U3")
@@
 		)
 		(instances
-			(project "ByggernProject"
+			(project "ByggernProject (2)"
 				(path "/43741492-b21a-4f5a-8ce1-a54a4b312e32"
 					(reference "U7")
@@
 		)
 		(instances
-			(project "ByggernProject"
+			(project "ByggernProject (2)"
 				(path "/43741492-b21a-4f5a-8ce1-a54a4b312e32"
 					(reference "#PWR016")
@@
 		)
 		(instances
-			(project "ByggernProject"
+			(project "ByggernProject (2)"
 				(path "/43741492-b21a-4f5a-8ce1-a54a4b312e32"
 					(reference "U6")
@@
 		)
 		(instances
-			(project "ByggernProject"
+			(project "ByggernProject (2)"
 				(path "/43741492-b21a-4f5a-8ce1-a54a4b312e32"
 					(reference "#PWR027")
@@
 		)
 		(instances
-			(project "ByggernProject"
+			(project "ByggernProject (2)"
 				(path "/43741492-b21a-4f5a-8ce1-a54a4b312e32"
 					(reference "SW2")
@@
 		)
 		(instances
-			(project "ByggernProject"
+			(project "ByggernProject (2)"
 				(path "/43741492-b21a-4f5a-8ce1-a54a4b312e32"
 					(reference "#PWR013")
@@
 		)
 		(instances
-			(project "ByggernProject"
+			(project "ByggernProject (2)"
 				(path "/43741492-b21a-4f5a-8ce1-a54a4b312e32"
 					(reference "0.1my")
@@
 		)
 		(instances
-			(project "ByggernProject"
+			(project "ByggernProject (2)"
 				(path "/43741492-b21a-4f5a-8ce1-a54a4b312e32"
 					(reference "U9")
@@
 		)
 		(instances
-			(project "ByggernProject"
+			(project "ByggernProject (2)"
 				(path "/43741492-b21a-4f5a-8ce1-a54a4b312e32"
 					(reference "#PWR07")
@@
 		)
 		(instances
-			(project "ByggernProject"
+			(project "ByggernProject (2)"
 				(path "/43741492-b21a-4f5a-8ce1-a54a4b312e32"
 					(reference "J2")
@@
 		)
 		(instances
-			(project "ByggernProject"
+			(project "ByggernProject (2)"
 				(path "/43741492-b21a-4f5a-8ce1-a54a4b312e32"
 					(reference "C6")
@@
 		)
 		(instances
-			(project "ByggernProject"
+			(project "ByggernProject (2)"
 				(path "/43741492-b21a-4f5a-8ce1-a54a4b312e32"
 					(reference "#PWR031")
@@
 		)
 		(instances
-			(project "ByggernProject"
+			(project "ByggernProject (2)"
 				(path "/43741492-b21a-4f5a-8ce1-a54a4b312e32"
 					(reference "#PWR015")
@@
 		)
 		(instances
-			(project "ByggernProject"
+			(project "ByggernProject (2)"
 				(path "/43741492-b21a-4f5a-8ce1-a54a4b312e32"
 					(reference "#PWR024")
@@
 		)
 		(instances
-			(project "ByggernProject"
+			(project "ByggernProject (2)"
 				(path "/43741492-b21a-4f5a-8ce1-a54a4b312e32"
 					(reference "#PWR012")
@@
 		)
 		(instances
-			(project "ByggernProject"
+			(project "ByggernProject (2)"
 				(path "/43741492-b21a-4f5a-8ce1-a54a4b312e32"
 					(reference "ADC")
@@
 		)
 		(instances
-			(project "ByggernProject"
+			(project "ByggernProject (2)"
 				(path "/43741492-b21a-4f5a-8ce1-a54a4b312e32"
 					(page "2")
