File: KiCad/sramblock.kicad_sch (KiCad schematic)
At the start: 2 parts, among them U4 LATCH, U8 SRAM

Commit message: Add files via upload
Parts:
- removed U4: LATCH, symbol 74xx:74LS573
- removed U8: SRAM, Package_SO:SOP-28_8.4x18.16mm_P1.27mm, symbol Memory_RAM:HY6264AxJ
